File: Schematic2/After-near-death-experience.kicad_pcb (KiCad board)
At the start: 2 copper layers, 8.5 x 71 mm, 52 parts, among them SW1 Rotary_Encoder_Switch, U1 Kailhlowprofile, U10 Kailhlowprofile, U11 Kailhlowprofile, U12 Kailhlowprofile, U13 Kailhlowprofile, U14 Kailhlowprofile, U15 Kailhlowprofile, U16 Kailhlowprofile, U17 Kailhlowprofile, U18 Kailhlowprofile, U19 Kailhlowprofile, U2 Kailhlowprofile, U20 Kailhlowprofile, U3 Kailhlowprofile, U4 Kailhlowprofile, U5 Kailhlowprofile, U6 Kailhlowprofile, U7 Kailhlowprofile, U8 Kailhlowprofile, U9 Kailhlowprofile

Commit message: The final countdown
The diamond deluxe of FINAL
Parts:
- moved D15 200.0 mm to (78.1, 87.2)
- moved Ard1 200.0 mm to (94.6, 19.9)
- moved D1 200.0 mm to (36.1, 27.9)
- moved D10 200.0 mm to (57.0, 67.3)
- moved D11 200.0 mm to (78.0, 67.3)
- moved D12 200.0 mm to (98.7, 67.3)
- moved D13 200.0 mm to (36.0, 87.2)
- moved D14 200.0 mm to (57.0, 87.2)
- moved D16 200.0 mm to (98.8, 87.2)
- moved D17 200.0 mm to (36.0, 107.0)
- moved D18 200.0 mm to (57.0, 107.0)
- moved D19 200.0 mm to (78.0, 107.0)
- moved D20 200.0 mm to (98.7, 107.0)
- moved D3 200.0 mm to (78.0, 27.7)
- moved D4 200.0 mm to (98.8, 27.6)
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Routing:
- net R5: track 0.00 -> 183.0 mm, vias 0 -> 7
- net R4: track 0.00 -> 161.5 mm, vias 0 -> 5
- net C1: track 0.00 -> 159.2 mm
- net C2: track 0.11 -> 140.9 mm
- net R3: track 0.00 -> 137.4 mm, vias 0 -> 3
- net C3: track 0.00 -> 122.8 mm
- net R2: track 0.00 -> 108.5 mm, vias 0 -> 1
- net C4: track 0.00 -> 108.5 mm
- net S1: track 0.00 -> 103.2 mm, vias 0 -> 2
- net R1: track 0.00 -> 96.2 mm
- net Net-(DI4-Pad2): track 0.00 -> 79.3 mm, vias 0 -> 2
- net Net-(DI1-Pad2): track 0.00 -> 69.0 mm, vias 0 -> 1
- net EnGNDC1: track 0.00 -> 49.8 mm, vias 0 -> 3
- net Net-(DI5-Pad2): track 0.00 -> 29.1 mm
- net Net-(D17-Pad2): track 0.00 -> 18.0 mm
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Other:
- board size 8.5 x 71 mm -> 100 x 119 mm
