File: Schematic2/Schematic2.kicad_pcb (KiCad board)
At the start: 2 copper layers, 100 x 119 mm, 52 parts, among them SW1 Rotary_Encoder_Switch, U1 Kailhlowprofile, U10 Kailhlowprofile, U11 Kailhlowprofile, U12 Kailhlowprofile, U13 Kailhlowprofile, U14 Kailhlowprofile, U15 Kailhlowprofile, U16 Kailhlowprofile, U17 Kailhlowprofile, U18 Kailhlowprofile, U19 Kailhlowprofile, U2 Kailhlowprofile, U20 Kailhlowprofile, U3 Kailhlowprofile, U4 Kailhlowprofile, U5 Kailhlowprofile, U6 Kailhlowprofile, U7 Kailhlowprofile, U8 Kailhlowprofile, U9 Kailhlowprofile

Commit message: The final countdown
The diamond deluxe of FINAL
Parts:
- Ard1: moved to B.Cu
- moved SW1 186.5 mm to (46.0, 40.5), turned to 180 degrees
- moved R1 180.8 mm to (33.0, 46.7), turned to 270 degrees
- moved U4 171.7 mm to (118.5, 57.5)
- moved U1 167.9 mm to (55.5, 57.5)
- moved D5 158.4 mm to (66.0, 77.0), turned to 90 degrees
- moved D8 152.7 mm to (128.8, 77.0), turned to 90 degrees
- moved D6 150.5 mm to (87.0, 77.0), turned to 90 degrees
- moved U2 149.2 mm to (76.5, 57.5)
- moved D3 143.5 mm to (107.9, 57.7), turned to 90 degrees
- moved D9 142.1 mm to (66.0, 97.3), turned to 90 degrees
- moved D4 137.3 mm to (128.7, 57.6), turned to 90 degrees
- moved DI1 135.6 mm to (44.5, 92.4), turned to 180 degrees
- moved D10 135.4 mm to (87.0, 97.3), turned to 90 degrees
- moved D1 134.6 mm to (66.0, 57.9), turned to 90 degrees
- moved D11 134.5 mm to (108.0, 97.3), turned to 90 degrees
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Connections:
- DI3 pad 2: Net-(DI3-Pad2) -> EnGNDC1
- DI7 pad 2: Net-(DI7-Pad2) -> S1
- S1 pad 1: Net-(DI7-Pad2) -> S1
- SW1 pad C: Net-(DI3-Pad2) -> EnGNDC1
Routing:
- net S1: track 0.00 -> 312.9 mm, vias 0 -> 6
- net EnGNDC1: track 0.00 -> 189.1 mm, vias 0 -> 6
- net R5: track 0.00 -> 183.0 mm, vias 0 -> 7
- net R4: track 0.00 -> 161.5 mm, vias 0 -> 5
- net C1: track 0.00 -> 159.2 mm
- net Net-(DI6-Pad2): track 0.00 -> 152.7 mm, vias 0 -> 4
- net EnPWMB: track 0.00 -> 142.8 mm, vias 0 -> 5
- net C2: track 0.00 -> 140.9 mm
- net R3: track 0.00 -> 137.4 mm, vias 0 -> 3
- net EnPWMA: track 0.00 -> 131.3 mm, vias 0 -> 6
- net C3: track 0.00 -> 122.8 mm
- net S2-2: track 0.00 -> 117.4 mm, vias 0 -> 4
- net S2: track 0.00 -> 115.5 mm, vias 0 -> 4
- net R2: track 0.00 -> 108.5 mm, vias 0 -> 1
- net C4: track 0.00 -> 108.5 mm
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Other:
- outline, holes or cut-outs redrawn
- net class Default: trace_width 0.25 -> 0.4
